File: electronics/power_control_pcb/power_control_pcb.kicad_pcb (KiCad board)
At the start: 2 copper layers, 108 x 55 mm, 89 parts, among them J1 +48V_FUSED, J2 48V_IN, J3 Status, J4 PGND_OUT, J5 +12V_OUT, J6 CURR_MONITOR, J7 Status_12V, J8 FET_OUT, J9 Control, Q1 IRF4905, Q2 PTD15N10, Q3 PTD15N10, Q4 PTD15N10, Q5 PTD15N10, U1 LTV-356T, U10 LTV-356T, U11 LTV-356T, U12 LTV-356T, U2 TL431ACDBZ, U3 ACS711xLCTR-12AB, U4 LTV-356T, U5 LTV-356T, U6 LTV-356T, U7 L78L05_SOT89, U8 LTV-356T, U9 SY8502

Commit message: Update wiring diagram & motor driver part values
Parts:
- turned D10 to 0 degrees
- turned D11 to 180 degrees
- turned D4 to 0 degrees
- turned D9 to 180 degrees
Connections:
- D10 pad 1: GND -> /FET2_DRAIN
- D10 pad 2: /FET2_DRAIN -> GND
- D11 pad 1: GND -> /FET1_DRAIN
- D11 pad 2: /FET1_DRAIN -> GND
- D4 pad 1: GND -> /+48V_FUSED
- D4 pad 2: /+48V_FUSED -> GND
- D9 pad 1: GND -> /FET3_DRAIN
- D9 pad 2: /FET3_DRAIN -> GND
Changed lines of the file:
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@@
   )
   (footprint "Diode_SMD:D_SMA" (layer "B.Cu")
-    (at 227.9 92.2)
+    (at 227.9 92.2 180)
     (descr "Diode SMA (DO-214AC)")
     (tags "Diode SMA (DO-214AC)")
@@
     (fp_line (start -2.3 -1.5) (end -2.3 1.5) (layer "B.Fab") (width 0.1))
     (fp_line (start -0.64944 -0.00102) (end 0.50118 -0.75032) (layer "B.Fab") (width 0.1))
-    (pad "1" smd rect locked (at -2 0) (size 2.5 1.8) (layers "B.Cu" "B.Paste" "B.Mask")
-      (net 2 "GND") (pinfunction "A1") (pintype "passive"))
-    (pad "2" smd rect locked (at 2 0) (size 2.5 1.8) (layers "B.Cu" "B.Paste" "B.Mask")
-      (net 19 "/FET1_DRAIN") (pinfunction "A2") (pintype "passive"))
+    (pad "1" smd rect locked (at -2 0 180) (size 2.5 1.8) (layers "B.Cu" "B.Paste" "B.Mask")
+      (net 19 "/FET1_DRAIN") (pinfunction "K") (pintype "passive"))
+    (pad "2" smd rect locked (at 2 0 180) (size 2.5 1.8) (layers "B.Cu" "B.Paste" "B.Mask")
+      (net 2 "GND") (pinfunction "A") (pintype "passive"))
     (model "${KICAD6_3DMODEL_DIR}/Diode_SMD.3dshapes/D_SMA.wrl"
       (offset (xyz 0 0 0))
@@
   )
   (footprint "Diode_SMD:D_SMA" (layer "B.Cu")
-    (at 220.4 92.2 180)
+    (at 220.4 92.2)
     (descr "Diode SMA (DO-214AC)")
     (tags "Diode SMA (DO-214AC)")
@@
     (fp_line (start -2.3 -1.5) (end -2.3 1.5) (layer "B.Fab") (width 0.1))
     (fp_line (start -0.64944 -0.00102) (end 0.50118 0.79908) (layer "B.Fab") (width 0.1))
-    (pad "1" smd rect locked (at -2 0 180) (size 2.5 1.8) (layers "B.Cu" "B.Paste" "B.Mask")
-      (net 2 "GND") (pinfunction "A1") (pintype "passive"))
-    (pad "2" smd rect locked (at 2 0 180) (size 2.5 1.8) (layers "B.Cu" "B.Paste" "B.Mask")
-      (net 18 "/FET2_DRAIN") (pinfunction "A2") (pintype "passive"))
+    (pad "1" smd rect locked (at -2 0) (size 2.5 1.8) (layers "B.Cu" "B.Paste" "B.Mask")
+      (net 18 "/FET2_DRAIN") (pinfunction "K") (pintype "passive"))
+    (pad "2" smd rect locked (at 2 0) (size 2.5 1.8) (layers "B.Cu" "B.Paste" "B.Mask")
+      (net 2 "GND") (pinfunction "A") (pintype "passive"))
     (model "${KICAD6_3DMODEL_DIR}/Diode_SMD.3dshapes/D_SMA.wrl"
       (offset (xyz 0 0 0))
@@
     (fp_line (start -0.64944 -0.00102) (end 0.50118 0.79908) (layer "B.Fab") (width 0.1))
     (pad "1" smd rect locked (at -2 0 180) (size 2.5 1.8) (layers "B.Cu" "B.Paste" "B.Mask")
-      (net 8 "+12V") (pinfunction "A1") (pintype "passive"))
+      (net 8 "+12V") (pinfunction "K") (pintype "passive"))
     (pad "2" smd rect locked (at 2 0 180) (size 2.5 1.8) (layers "B.Cu" "B.Paste" "B.Mask")
-      (net 2 "GND") (pinfunction "A2") (pintype "passive"))
+      (net 2 "GND") (pinfunction "A") (pintype "passive"))
     (model "${KICAD6_3DMODEL_DIR}/Diode_SMD.3dshapes/D_SMA.wrl"
       (offset (xyz 0 0 0))
@@
   )
   (footprint "Diode_SMD:D_SMA" (layer "B.Cu")
-    (at 165.9 90.7 180)
+    (at 165.9 90.7)
     (descr "Diode SMA (DO-214AC)")
     (tags "Diode SMA (DO-214AC)")
@@
     (fp_line (start -2.3 -1.5) (end -2.3 1.5) (layer "B.Fab") (width 0.1))
     (fp_line (start 0.50118 -0.00102) (end 1.4994 -0.00102) (layer "B.Fab") (width 0.1))
-    (pad "1" smd rect locked (at -2 0 180) (size 2.5 1.8) (layers "B.Cu" "B.Paste" "B.Mask")
-      (net 2 "GND") (pinfunction "A1") (pintype "passive"))
-    (pad "2" smd rect locked (at 2 0 180) (size 2.5 1.8) (layers "B.Cu" "B.Paste" "B.Mask")
-      (net 1 "/+48V_FUSED") (pinfunction "A2") (pintype "passive"))
+    (pad "1" smd rect locked (at -2 0) (size 2.5 1.8) (layers "B.Cu" "B.Paste" "B.Mask")
+      (net 1 "/+48V_FUSED") (pinfunction "K") (pintype "passive"))
+    (pad "2" smd rect locked (at 2 0) (size 2.5 1.8) (layers "B.Cu" "B.Paste" "B.Mask")
+      (net 2 "GND") (pinfunction "A") (pintype "passive"))
     (model "${KICAD6_3DMODEL_DIR}/Diode_SMD.3dshapes/D_SMA.wrl"
       (offset (xyz 0 0 0))
@@
   )
   (footprint "Diode_SMD:D_SMA" (layer "B.Cu")
-    (at 213 92.2)
+    (at 213 92.2 180)
     (descr "Diode SMA (DO-214AC)")
     (tags "Diode SMA (DO-214AC)")
@@
     (fp_line (start 0.50118 -0.00102) (end 1.4994 -0.00102) (layer "B.Fab") (width 0.1))
     (fp_line (start 2.3 1.5) (end -2.3 1.5) (layer "B.Fab") (width 0.1))
-    (pad "1" smd rect locked (at -2 0) (size 2.5 1.8) (layers "B.Cu" "B.Paste" "B.Mask")
-      (net 2 "GND") (pinfunction "A1") (pintype "passive"))
-    (pad "2" smd rect locked (at 2 0) (size 2.5 1.8) (layers "B.Cu" "B.Paste" "B.Mask")
-      (net 17 "/FET3_DRAIN") (pinfunction "A2") (pintype "passive"))
+    (pad "1" smd rect locked (at -2 0 180) (size 2.5 1.8) (layers "B.Cu" "B.Paste" "B.Mask")
+      (net 17 "/FET3_DRAIN") (pinfunction "K") (pintype "passive"))
+    (pad "2" smd rect locked (at 2 0 180) (size 2.5 1.8) (layers "B.Cu" "B.Paste" "B.Mask")
+      (net 2 "GND") (pinfunction "A") (pintype "passive"))
     (model "${KICAD6_3DMODEL_DIR}/Diode_SMD.3dshapes/D_SMA.wrl"
       (offset (xyz 0 0 0))
